Commit message: [description] Generalization. Add unit test using kobuki.
[description][test] Use source permission to pass the tests in install space.

File: openni_description/model/kinect.urdf.xacro (robot description, xacro)
@@ -1,11 +1,9 @@
 <?xml version="1.0"?>
-<robot name="sensor_kinect" xmlns:xacro="http://ros.org/wiki/xacro">
-  <xacro:include filename="$(find turtlebot_description)/urdf/turtlebot_gazebo.urdf.xacro"/>
-  <xacro:include filename="$(find turtlebot_description)/urdf/turtlebot_properties.urdf.xacro"/>
-  <xacro:property name="kinect_cam_py" value="-0.0125"/>
+<robot name="sensor_openni" xmlns:xacro="http://ros.org/wiki/xacro">
+  <xacro:include filename="$(find openni_description)/model/kinect_gazebo.urdf.xacro" />
   <!-- Parameterised in part by the values in turtlebot_properties.urdf.xacro -->
-  <xacro:macro name="sensor_kinect" params="parent">
+  <xacro:macro name="sensor_kinect" params="parent cam_px cam_py cam_pz cam_or cam_op cam_oy">
     <joint name="camera_rgb_joint" type="fixed">
-      <origin xyz="${cam_px} ${kinect_cam_py} ${cam_pz}" rpy="${cam_or} ${cam_op} ${cam_oy}"/>
+      <origin xyz="${cam_px} ${cam_py} ${cam_pz}" rpy="${cam_or} ${cam_op} ${cam_oy}"/>
       <parent link="${parent}"/>
       <child link="camera_rgb_frame" />
@@ -19,5 +17,5 @@
     <link name="camera_rgb_optical_frame"/>
     <joint name="camera_joint" type="fixed">
-      <origin xyz="-0.031 ${-kinect_cam_py} -0.016" rpy="0 0 0"/>
+      <origin xyz="-0.031 ${-cam_py} -0.016" rpy="0 0 0"/>
       <parent link="camera_rgb_frame"/>
       <child link="camera_link"/>
@@ -27,5 +25,5 @@
        <origin xyz="0 0 0" rpy="0 0 ${M_PI/2}"/>
         <geometry>
-         <mesh filename="package://turtlebot_description/meshes/sensors/kinect.dae"/>
+         <mesh filename="package://openni_description/mesh/kinect.dae"/>
         </geometry>
       </visual>
@@ -48,5 +46,5 @@
          (Hence, don't publish them additionally!) -->
 	<joint name="camera_depth_joint" type="fixed">
-	  <origin xyz="0 ${2 * -kinect_cam_py} 0" rpy="0 0 0" />
+	  <origin xyz="0 ${2 * -cam_py} 0" rpy="0 0 0" />
 	  <parent link="camera_rgb_frame" />
 	  <child link="camera_depth_frame" />
@@ -60,5 +58,5 @@
 	<link name="camera_depth_optical_frame"/>
 	<!-- Kinect sensor for simulation -->
-	<turtlebot_sim_3dsensor/>
+	<sim_3dsensor_kinect/>
   </xacro:macro>
 </robot>

File: openni_description/test/turtlebot_properties.urdf.xacro (robot description, xacro)
@@ -20,5 +20,5 @@
    -->
 	<xacro:property name="cam_px" value="-0.087" />
-<!--	<xacro:property name="cam_py" value="-0.0125" /> Y varies for different configurations. get sets in sensors_urdf -->
+        <xacro:property name="cam_py" value="-0.0125"/>
 	<xacro:property name="cam_pz" value="0.2870" />
 	<xacro:property name="cam_or" value="0" />
